Commit message: [upadte]動くロボット実装

File: sim1_lecture/xacro/dtw_robot1.xacro (robot description, xacro)
@@ -2,8 +2,8 @@
 <robot name="dtw_robot" xmlns:xacro="http://ros.org/wiki/xacro">
   <material name="gray">
-    <color rgba="0.5 0.5 0.5 2.5"/>
+    <color rgba="0.5 0.5 0.5 1"/>
   </material>
   <material name="red">
-    <color rgba="1.0 0.0 0.0 2.5"/>
+    <color rgba="1.0 0.0 0.0 1"/>
   </material>
   <xacro:macro name="wheel_macro" params="parent prefix xyz">

File: sim1_lecture/xacro/dtw_robot2.xacro (robot description, xacro)
@@ -2,8 +2,8 @@
 <robot name="dtw_robot" xmlns:xacro="http://ros.org/wiki/xacro">
   <material name="gray">
-    <color rgba="0.5 0.5 0.5 2.5"/>
+    <color rgba="0.5 0.5 0.5 1"/>
   </material>
   <material name="red">
-    <color rgba="1.0 0.0 0.0 2.5"/>
+    <color rgba="1.0 0.0 0.0 1"/>
   </material>
   <xacro:macro name="wheel_macro" params="parent prefix xyz">

File: sim1_lecture/xacro/dtw_robot3.xacro (robot description, xacro)
@@ -2,8 +2,8 @@
 <robot name="dtw_robot" xmlns:xacro="http://ros.org/wiki/xacro">
   <material name="gray">
-    <color rgba="0.5 0.5 0.5 2.5"/>
+    <color rgba="0.5 0.5 0.5 1"/>
   </material>
   <material name="red">
-    <color rgba="1.0 0.0 0.0 2.5"/>
+    <color rgba="1.0 0.0 0.0 1"/>
   </material>
   <xacro:macro name="wheel_macro" params="parent prefix xyz">
@@ -101,4 +101,26 @@
     </collision>
   </link>
+  <xacro:property name="height" value="1.2" />
+  <joint name="center_pillar" type="fixed">
+    <parent link="base_link"/>
+    <child  link="center_pillar_link"/>
+    <origin xyz="0 0 ${height/2+0.1}" rpy="0 0 0"/>
+  </joint>
+  <link name="center_pillar_link">
+    <visual>
+      <origin xyz="0 0 0" rpy="0 0 0" />
+      <geometry>
+        <box size="0.1 0.1 ${height}" />
+      </geometry>
+      <material name="gray" />
+    </visual>
+    <collision>
+      <origin xyz="0 0 0" rpy="0 0 0" />
+      <geometry>
+        <box size="0.1 0.1 ${height}" />
+      </geometry>
+      <material name="gray" />
+    </collision>
+  </link>
   <gazebo reference="ball_link">
     <material>Gazebo/Gray</material>

File: vis_lecture/xacro/basic3.xacro (robot description, xacro)
@@ -1,9 +1,9 @@
 <robot name="test_robot" xmlns:xacro="http://ros.org/wiki/xacro">
-  <xacro:property name="color" value="blue" />
+  <xacro:property name="color" value="red" />
   <material name="red">
-    <color rgba="1.0 0.0 0.0 2.0"/>
+    <color rgba="1.0 0.0 0.0 1"/>
   </material>
   <material name="blue">
-    <color rgba="0.0 0.0 1.0 2.0"/>
+    <color rgba="0.0 0.0 1.0 1"/>
   </material>
   <link name="base_link">
